Commit message: Changed transimision to effort controllers, added xacro tags for sensors noetic compatibility and corrected issue with materials moving the conflicting materials to a separate xacro file

File: urdf/all_sensors.urdf.xacro (robot description, xacro)
@@ -4,4 +4,6 @@
   <xacro:include filename="$(find robotnik_sensors)/urdf/utils/inertia.urdf.xacro" />
   <!-- This file unifies all sensors that can be used on simulation, defined as xacro:macros -->
+  <!-- Common Materials -->
+  <xacro:include filename="$(find robotnik_sensors)/urdf/materials.xacro" />
   <!-- Axis p5512 -->
   <xacro:include filename="$(find robotnik_sensors)/urdf/axis.urdf.xacro" />

File: urdf/axis_q8641.urdf.xacro (robot description, xacro)
@@ -73,8 +73,10 @@
       <type>transmission_interface/SimpleTransmission</type>
       <joint name="${prefix}_pan_joint">
-        <hardwareInterface>hardware_interface/VelocityJointInterface</hardwareInterface>
+        <hardwareInterface>hardware_interface/EffortJointInterface</hardwareInterface>
+        <!-- <hardwareInterface>hardware_interface/VelocityJointInterface</hardwareInterface> -->
       </joint>
       <actuator name="pan_motor">
-        <hardwareInterface>hardware_interface/VelocityJointInterface</hardwareInterface>
+        <hardwareInterface>hardware_interface/EffortJointInterface</hardwareInterface>
+        <!-- <hardwareInterface>hardware_interface/VelocityJointInterface</hardwareInterface> -->
         <mechanicalReduction>${ptz_mechanical_reduction}</mechanicalReduction>
       </actuator>
@@ -115,8 +117,10 @@
       <type>transmission_interface/SimpleTransmission</type>
       <joint name="${prefix}_tilt_joint">
-        <hardwareInterface>hardware_interface/VelocityJointInterface</hardwareInterface>
+        <hardwareInterface>hardware_interface/EffortJointInterface</hardwareInterface>
+        <!-- <hardwareInterface>hardware_interface/VelocityJointInterface</hardwareInterface> -->
       </joint>
       <actuator name="tilt_motor">
-        <hardwareInterface>hardware_interface/VelocityJointInterface</hardwareInterface>
+        <hardwareInterface>hardware_interface/EffortJointInterface</hardwareInterface>
+        <!-- <hardwareInterface>hardware_interface/VelocityJointInterface</hardwareInterface> -->
         <mechanicalReduction>${ptz_mechanical_reduction}</mechanicalReduction>
       </actuator>
@@ -151,5 +155,5 @@
     </gazebo>
     <!-- Axis sensor for simulation -->
-    <sensor_axis_q8641_gazebo/>
+    <xacro:sensor_axis_q8641_gazebo/>
   </xacro:macro>
   <xacro:macro name="sensor_axis_q8641_gazebo">

File: urdf/benewake_ce30.urdf.xacro (robot description, xacro)
@@ -3,7 +3,4 @@
   <xacro:property name="M_PI" value="3.1415926535897931" />
   <xacro:macro name="sensor_benewake_ce30" params="prefix parent prefix_topic *origin range_min range_max hfov vfov fps gpu:=^|true">
-    <material name="black_alu">
-      <color rgba="0.9 0.9 0.9 1"/>
-    </material>
     <joint name="${prefix}_base_joint" type="fixed">
       <xacro:insert_block name="origin" />

File: urdf/benewake_ce30d.urdf.xacro (robot description, xacro)
@@ -3,7 +3,4 @@
   <xacro:property name="M_PI" value="3.1415926535897931" />
   <xacro:macro name="sensor_benewake_ce30d" params="prefix parent prefix_topic:='lidar_3d' *origin range_min:=0.4 range_max:=28.0 hfov:=60.0 vfov:=4.0 fps:=30.0 gpu:=^|true">
-    <material name="black_alu">
-      <color rgba="0.9 0.9 0.9 1"/>
-    </material>
     <joint name="${prefix}_base_joint" type="fixed">
       <xacro:insert_block name="origin" />
@@ -40,5 +37,5 @@
     </joint>
     <link name="${prefix}_link"/>
-  <sensor_benewake_ce30d_gazebo range_min="${range_min}" range_max="${range_max}" hfov="${hfov}" vfov="${vfov}" fps="${fps}" gpu="${gpu}"/>
+  <xacro:sensor_benewake_ce30d_gazebo range_min="${range_min}" range_max="${range_max}" hfov="${hfov}" vfov="${vfov}" fps="${fps}" gpu="${gpu}"/>
   </xacro:macro>
   <xacro:macro name="sensor_benewake_ce30d_gazebo" params="range_min range_max hfov vfov fps gpu">
@@ -51,5 +48,5 @@
       <xacro:unless value="${gpu}">
         <xacro:property name="ray_type" value="ray" />
-        <xacro:property name="plugin_lib" value="libgazebo_ros_block_laser.so" />
+        <xacro:property name="plugin_lib" value="libgazebo_ros_velodyne_laser.so" />
       </xacro:unless>
         <sensor type="${ray_type}" name="${prefix}_sensor">

File: urdf/hokuyo_utm30lx.urdf.xacro (robot description, xacro)
@@ -32,5 +32,5 @@
 	</joint>
     <!-- Hokuyo sensor for simulation -->
-    <sensor_hokuyo_utm_gazebo/>
+    <xacro:sensor_hokuyo_utm_gazebo/>
   </xacro:macro>
   <xacro:macro name="sensor_hokuyo_utm_gazebo">

File: urdf/ouster1.urdf.xacro (robot description, xacro)
@@ -3,7 +3,4 @@
   <xacro:property name="M_PI" value="3.1415926535897931" />
   <xacro:macro name="sensor_ouster1" params="prefix parent prefix_topic *origin range_min range_max hfov hsamples vfov vsamples fps gpu:=^|true">
-    <material name="black_alu">
-      <color rgba="0.9 0.9 0.9 1"/>
-    </material>
     <joint name="${prefix}_base_joint" type="fixed">
       <xacro:insert_block name="origin" />

File: urdf/rslidar.urdf.xacro (robot description, xacro)
@@ -2,8 +2,5 @@
 <robot name="sensor_rslidar" xmlns:xacro="http://wiki.ros.org/xacro">
   <xacro:property name="M_PI" value="3.1415926535897931" />
-  <xacro:macro name="sensor_rslidar" params="prefix parent prefix_topic *origin range_min range_max hfov hres vfov vres fps gpu:=^|true">
-    <material name="black_alu">
-      <color rgba="0.9 0.9 0.9 1"/>
-    </material>
+  <xacro:macro name="sensor_rslidar" params="prefix parent prefix_topic *origin range_min range_max hfov hres vfov vres fps gpu:=true">
     <joint name="${prefix}_base_joint" type="fixed">
       <xacro:insert_block name="origin" />
@@ -38,5 +35,5 @@
     </joint>
     <link name="${prefix}_link"/>
-  <sensor_rslidar_gazebo range_min="${range_min}" range_max="${range_max}" hfov="${hfov}" hres="${hres}" vfov="${vfov}" vres="${vres}" fps="${fps}" gpu="${gpu}"/>
+    <xacro:sensor_rslidar_gazebo range_min="${range_min}" range_max="${range_max}" hfov="${hfov}" hres="${hres}" vfov="${vfov}" vres="${vres}" fps="${fps}" gpu="${gpu}"/>
   </xacro:macro>
   <xacro:macro name="sensor_rslidar_gazebo" params="range_min range_max hfov hres vfov vres fps gpu">

File: urdf/rslidar_mems.urdf.xacro (robot description, xacro)
@@ -3,7 +3,4 @@
   <xacro:property name="M_PI" value="3.1415926535897931" />
   <xacro:macro name="sensor_rslidar_mems" params="prefix parent *origin">
-    <material name="black_alu">
-      <color rgba="0.9 0.9 0.9 1"/>
-    </material>
     <joint name="${prefix}_base_joint" type="fixed">
       <xacro:insert_block name="origin" />

Commit message: Added new camera from bosh MPC3 and added some adaptations for noetic XACRO limitations

File: urdf/all_sensors.urdf.xacro (robot description, xacro)
@@ -101,3 +101,5 @@
   <!-- Orbbec Embedded S -->
   <xacro:include filename="$(find robotnik_sensors)/urdf/embedded_s.urdf.xacro" />
+  <!-- Bosh Autonomous Driving Camera -->
+  <xacro:include filename="$(find robotnik_sensors)/urdf/mpc3_bosch.urdf.xacro" />
 </robot>

File: urdf/axis_q8641.urdf.xacro (robot description, xacro)
@@ -15,7 +15,7 @@
     <link name="${prefix}_base_link">
       <inertial>
-        <mass value="2"/>
+        <mass value="0.1"/>
         <origin xyz="0 0 0.06" rpy="0 0 0"/>
-        <xacro:solid_cuboid_inertia m="2" w="0.175" h="0.175" d="0.12" />
+        <xacro:solid_cuboid_inertia m="0.1" w="0.175" h="0.175" d="0.12" />
       </inertial>
       <visual>
@@ -48,7 +48,7 @@
     <link name="${prefix}_pan_link">
       <inertial>
-        <mass value="5.0"/>
+        <mass value="0.1"/>
         <origin xyz="0 0 0.12" rpy="0 0 0"/>
-        <xacro:solid_cuboid_inertia m="5.0" w="0.175" h="0.175" d="0.24" />
+        <xacro:solid_cuboid_inertia m="0.1" w="0.175" h="0.175" d="0.24" />
       </inertial>
       <visual>
@@ -92,7 +92,7 @@
     <link name="${prefix}_tilt_link">
       <inertial>
-        <mass value="5.0"/>
+        <mass value="0.1"/>
         <origin xyz="0.04875 0 0.11" rpy="0 0 0"/>
-        <xacro:solid_cuboid_inertia m="5.0" w="0.24" h="0.09" d="0.09" />
+        <xacro:solid_cuboid_inertia m="0.1" w="0.24" h="0.09" d="0.09" />
       </inertial>
       <visual>

File: urdf/benewake_ce30d.urdf.xacro (robot description, xacro)
@@ -19,5 +19,5 @@
       </visual>
       <collision>
-        <origin xyz="0 0 0" rpy="0 0 0"/>
+        <origin xyz="0 0 0" rpy="1.5708 0 1.5708"/>
         <geometry>
           <mesh filename="package://robotnik_sensors/meshes/benewake_ce30d.stl" />

File: urdf/mpc3_bosch.urdf.xacro (robot description, xacro)
@@ -1,5 +1,5 @@
 <?xml version="1.0"?>
 <robot xmlns:xacro="http://wiki.ros.org/xacro">
-  <xacro:macro name="sensor_ueye_cp_gige" params="prefix parent *origin">
+  <xacro:macro name="sensor_mpc3_bosch" params="prefix parent *origin">
     <joint name="${prefix}_joint" type="fixed">
       <xacro:insert_block name="origin"/>
@@ -55,20 +55,20 @@
     </inertial>
     </link>
-    <xacro:sensor_ueye_cp_gige_gazebo />
+    <xacro:sensor_mpc3_bosch_gazebo />
   </xacro:macro>
-  <xacro:macro name="sensor_ueye_cp_gige_gazebo">
+  <xacro:macro name="sensor_mpc3_bosch_gazebo">
     <gazebo reference="${prefix}_base_link">
       <sensor type="camera" name="${prefix}_sensor">
         <update_rate>30.0</update_rate>
         <camera name="head">
-          <horizontal_fov>1.3962634</horizontal_fov>
+          <horizontal_fov>1.74</horizontal_fov>
           <image>
-            <width>800</width>
-            <height>800</height>
+            <width>640</width>
+            <height>480</height>
             <format>R8G8B8</format>
           </image>
           <clip>
             <near>0.03</near>
-            <far>300</far>
+            <far>160.0</far>
           </clip>
           <noise>
